File: Smart_Farm/Smart_Farm.kicad_sch (KiCad schematic)
At the start: 23 parts, among them J1 EJ508A, J2 Screw_Terminal_01x03, Q1 2N3904, U1 ESP32-DEVKITC-32D, U2 LCD 16x2 I2C, U3 SOIL SENSOR, U4 RTC, U5 Relay Module

Commit message: Update Schematic and PCB
Parts:
- removed SENS-1: DHT11, Smart_Farm:SENSOR-DHT11, symbol Smart_Farm:DHT11
- added C1: C_Polarized_Small_US, Capacitor_SMD:CP_Elec_8x10.5, symbol Device:C_Polarized_Small_US
- added C2: C_Polarized_Small_US, Capacitor_SMD:CP_Elec_6.3x5.4, symbol Device:C_Polarized_Small_US
- added DHT1: DHT11, Connector_PinSocket_2.54mm:PinSocket_1x03_P2.54mm_Vertical, symbol Smart_Farm:DHT11
- added H1, H2: MountingHole, MountingHole:MountingHole_3.2mm_M3_ISO14580, symbol Mechanical:MountingHole
- added LM7805CT2: LM7805CT, Smart_Farm:LM7805CT, symbol Smart_Farm:LM7805CT
- added RAIN_SENSOR1: RAIN SENSOR, Connector_PinSocket_2.54mm:PinSocket_1x04_P2.54mm_Horizontal, symbol Smart_Farm:RAIN_SENSOR
- added S4: 100SP1T1B4M2QE, Smart_Farm:SW_100SP1T1B4M2QE, symbol Smart_Farm:100SP1T1B4M2QE
- R1, R2, R3, R4, R5: value 1k -> R
- renumbered S1 to BTN_LED1, S3 to BTN_Mode1, S2 to BTN_Pump1, D2 to D1, U1 to ESP32-DEVKITC-32D3, U2 to LCD16x2I2C2, D1 to LED1, U4 to RTC1, U5 to Relay_Module1, U3 to SOIL_SENSOR1
Connections:
- net +5V: now also C2.1, DHT1.1 (VCC), LM7805CT2.3 (OUT), RAIN_SENSOR1.1 (VCC); no longer F1.1
- net GND: now also C1.2, C2.2, DHT1.3 (GND), LM7805CT2.2 (GND), RAIN_SENSOR1.4 (GND)
- net IO_04: now also BTN_LED1.2; no longer LED1.2 (A)
- net IO_14: now also DHT1.2 (DAT)
- net IO_33: now also SOIL_SENSOR1.1 (AO); no longer BTN_LED1.2
- net at F1.2: now also S4.3; no longer J1.1
- net +12V: now reaches J2.2 (Pin_2), Relay_Module1.COM
- net +12V: now also F1.1, C1.1, LM7805CT2.1 (IN)
- net IO_27: now reaches ESP32-DEVKITC-32D3.J2-11 (IO27)
- net IO_27: now also RAIN_SENSOR1.3 (DO)
- net IO_13: now reaches ESP32-DEVKITC-32D3.J2-15 (IO13)
- net IO_13: now also R4.1
- net IO_18: now reaches ESP32-DEVKITC-32D3.J3-9 (IO18)
- net IO_18: now also LED1.2 (A)
- net IO_26: no longer names the net of ESP32-DEVKITC-32D3.J2-10 (IO26)
- net IO_26: no longer R4.1
- net IO_34: no longer names the net of ESP32-DEVKITC-32D3.J2-5 (IO34)
- net IO_34: no longer SOIL_SENSOR1.1 (AO)
- new net: J1.1, S4.2
Other:
- moved on the sheet: BTN_LED1, BTN_Mode1, BTN_Pump1, D1, D3, D4, D5, ESP32-DEVKITC-32D3, F1, J1, LCD16x2I2C2, LED1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

Commit message: Update files
Parts:
- removed D4, LED1: LED, LED_SMD:LED_0805_2012Metric, symbol Device:LED
- removed R1: R, Resistor_SMD:R_0805_2012Metric, symbol Device:R
- removed S4: 100SP1T1B4M2QE, Smart_Farm:SW_100SP1T1B4M2QE, symbol Smart_Farm:100SP1T1B4M2QE
- added D4: WS2812B, LED_SMD:LED_WS2812B_PLCC4_5.0x5.0mm_P3.2mm, symbol LED:WS2812B
- added SW1: MK-12C02-G020, Smart_Farm:MK-12C02-G020_GSW, symbol Smart_Farm:MK-12C02-G020
- C1: value C_Polarized_Small_US -> 470uF
- C2: value C_Polarized_Small_US -> 100uF
- R2, R3, R4: value R -> 1k
- R5: value R -> 10k
Connections:
- net +12V: no longer J2.2 (Pin_2), Relay_Module1.COM
- net +5V: now also D3.1 (K), RTC1.4 (VCC), Relay_Module1.A2, SOIL_SENSOR1.1 (VCC), D4.1 (VDD); no longer R5.2, RTC1.2 (VCC), SOIL_SENSOR1.4 (VCC)
- net GND: now also J2.1 (Pin_1), R5.1, RAIN_SENSOR1.2 (GND), RTC1.5 (GND), Relay_Module1.NO, SOIL_SENSOR1.2 (GND), D4.3 (VSS), SW1.4, SW1.5, SW1.6, SW1.7; no longer J1.3, Q1.1 (E), RAIN_SENSOR1.4 (GND), RTC1.1 (GND), SOIL_SENSOR1.3 (GND)
- net IO_18: now also D4.4 (DIN)
- net IO_22: now also RTC1.2 (SCL); no longer RTC1.4 (SCL)
- net IO_33: now also SOIL_SENSOR1.4 (AO); no longer SOIL_SENSOR1.1 (AO)
- net at F1.2: now also SW1.1
- net +12V Power: now reaches J1.1
- net +12V Power: now also J2.2 (Pin_2), Relay_Module1.COM, SW1.2
- new net: Q1.1 (E), R5.2
- no-connect marks 0 -> 35
Other:
- note added: "BUTTON"
- note added: "POWER"
- note added: "RELAY MODULE"
- note added: "SENSOR"
- note added: "VOLTAGE REDUCTION"
- moved on the sheet: BTN_LED1, BTN_Mode1, BTN_Pump1, C1, C2, D1, D3, DHT1, ESP32-DEVKITC-32D3, F1, H1, H2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

Commit message: Update images
Other:
- note added: "POWER IC"
- note removed: "VOLTAGE REDUCTION"
Changed lines of the file:
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@@
 			(font
 				(size 3.81 3.81)
-				(thickness 0.508)
+				(thickness 0.762)
 				(bold yes)
 			)
 		)
 	)
-	(text "VOLTAGE REDUCTION"
+	(text "POWER IC"
 		(exclude_from_sim no)
 		(at 146.812 20.32 0)
@@
 			(font
 				(size 3.81 3.81)
-				(thickness 0.254)
+				(thickness 0.762)
 				(bold yes)
 			)
@@
 		(on_board yes)
 		(dnp no)
-		(fields_autoplaced yes)
 		(property "Reference" "LCD16x2I2C2"
-			(at 162.56 81.2799 0)
-			(effects
-				(font
+			(at 145.034 75.184 0)
+			(effects
+				(font
